File: ELE_MB_A1.kicad_pcb (KiCad board)
At the start: 2 copper layers, 80 x 56 mm, 126 parts, among them J101 Conn_01x02, J102 Conn_01x02, J103 Conn_01x02, J104 Conn_01x02, J105 Conn_01x02, J106 Conn_01x02, J107 Conn_01x04, J108 Conn_01x03, J109 Conn_01x04, J110 Conn_01x03, J111 Conn_01x04, J112 Conn_01x04, J113 Conn_01x03, J114 Conn_01x04, J115 Conn_01x03, J116 Conn_01x04, J117 Conn_01x03, J118 Conn_01x03, J119 Conn_01x04, J120 Conn_01x03, J121 Conn_01x03, Q101 2N7002, Q102 SI2301CDS-T1-GE3, Q103 2N7002, Q104 2N7002, Q105 2N7002, Q106 2N7002, U101 TPS54302, U102 TPS54302, U103 SN65HVD230, U104 SN74LVC1T45DBV, U105 SN74LVC1T45DBV, U106 XIAO-ESP32-C3-DIP

Commit message: Finished board
Parts:
- added D105: B5818WS, PCM_JLCPCB:D_SOD-323, F.Cu at (146.2, 61.0)
- moved R140 5.04 mm to (109.1, 60.0), turned to 180 degrees
- moved R149 5.04 mm to (116.1, 60.0), turned to 180 degrees
- moved R137 5.02 mm to (105.6, 60.0), turned to 180 degrees
- moved R138 5.02 mm to (105.6, 65.0), turned to 180 degrees
- moved R141 5.02 mm to (109.1, 65.0), turned to 180 degrees
- moved R146 5.02 mm to (112.6, 60.0), turned to 180 degrees
- moved R147 5.02 mm to (112.6, 65.0), turned to 180 degrees
- moved R150 5.02 mm to (115.1, 65.0)
- moved R120 4.93 mm to (129.2, 62.2)
- moved R128 4.88 mm to (138.7, 62.2)
- moved D104 3.58 mm to (143.1, 63.5), turned to -90 degrees
- moved R114 3.40 mm to (142.7, 60.3)
- moved R123 3.31 mm to (127.3, 62.2), turned to 0 degrees
- moved R131 3.27 mm to (136.8, 62.2), turned to 0 degrees
- moved R102 2.90 mm to (140.7, 77.1)
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Connections:
- C114 pad 1: Net-(J106-Pin_2) -> Net-(C114-Pad1)
- J113 pad 1: Net-(J113-Pin_1) -> GND
- J113 pad 3: GND -> Net-(J113-Pin_3)
- J115 pad 1: Net-(J115-Pin_1) -> GND
- J115 pad 3: GND -> Net-(J115-Pin_3)
- J118 pad 1: Net-(J118-Pin_1) -> GND
- J118 pad 3: GND -> Net-(J118-Pin_3)
- J120 pad 1: Net-(J120-Pin_1) -> GND
- J120 pad 3: GND -> Net-(J120-Pin_3)
- J121 pad 1: Net-(J121-Pin_1) -> GND
- J121 pad 3: GND -> Net-(J121-Pin_3)
- JP102 pad JP1_1: /CAND -> unconnected-(JP102A-N17-PadJP1_1)
- JP102 pad JP1_10: unconnected-(JP102A-Y19-PadJP1_10) -> /LEDS
- JP102 pad JP1_19: unconnected-(JP102A-V16-PadJP1_19) -> /CANR
- JP102 pad JP1_2: /CANR -> unconnected-(JP102A-P18-PadJP1_2)
- JP102 pad JP1_21: unconnected-(JP102A-T17-PadJP1_21) -> /CAND
- JP102 pad JP1_3: unconnected-(JP102A-R16-PadJP1_3) -> /LIDAR_RX1
- JP102 pad JP1_5: /LIDAR_RX1 -> /LIDAR_RX2
- JP102 pad JP1_7: /LIDAR_RX2 -> /LIDAR_RX3
- JP102 pad JP1_8: /LIDAR_RX3 -> unconnected-(JP102A-W19-PadJP1_8)
- JP102 pad JP2_1: /SERVO2 -> /SERVO1
- JP102 pad JP2_10: /LIDAR_RX2 -> unconnected-(JP102B-A20-PadJP2_10)
- JP102 pad JP2_13: unconnected-(JP102B-D19-PadJP2_13) -> /AX_DIR2
- JP102 pad JP2_14: /SPARE26 -> unconnected-(JP102B-D20-PadJP2_14)
- JP102 pad JP2_16: /SPARE22 -> unconnected-(JP102B-D18-PadJP2_16)
- JP102 pad JP2_17: unconnected-(JP102B-H16-PadJP2_17) -> /AX_DATA2
- JP102 pad JP2_18: /SPARE21 -> unconnected-(JP102B-H17-PadJP2_18)
- JP102 pad JP2_19: /AX_DATA -> /AU
- JP102 pad JP2_2: /SERVO1 -> /WIFI_UART_RX
- JP102 pad JP2_20: /SPARE27 -> unconnected-(JP102B-G20-PadJP2_20)
- JP102 pad JP2_21: /AU -> unconnected-(JP102B-J18-PadJP2_21)
- JP102 pad JP2_22: /IO6 -> unconnected-(JP102B-H18-PadJP2_22)
- JP102 pad JP2_24: /IO4 -> unconnected-(JP102B-J16-PadJP2_24)
- JP102 pad JP2_26: /IO2 -> unconnected-(JP102B-B20-PadJP2_26)
- JP102 pad JP2_27: unconnected-(JP102B-G17-PadJP2_27) -> /TIRETTE
- JP102 pad JP2_28: /DIR1 -> unconnected-(JP102B-G18-PadJP2_28)
- JP102 pad JP2_3: /SERVO4 -> /SERVO3
- JP102 pad JP2_32: /STP1 -> unconnected-(JP102B-L20-PadJP2_32)
- JP102 pad JP2_33: /TIRETTE -> unconnected-(JP102B-F19-PadJP2_33)
- JP102 pad JP2_34: /DIR2 -> unconnected-(JP102B-F20-PadJP2_34)
- JP102 pad JP2_36: /nEN_DRIVER2 -> unconnected-(JP102B-M20-PadJP2_36)
- JP102 pad JP2_4: /SERVO3 -> /SERVO2
- JP102 pad JP2_40: /AX_DIR -> unconnected-(JP102B-H20-PadJP2_40)
- JP102 pad JP2_5: unconnected-(JP102B-F16-PadJP2_5) -> /WIFI_UART_TX
- JP102 pad JP2_6: /SERVO6 -> /SERVO4
- JP102 pad JP2_7: unconnected-(JP102B-E18-PadJP2_7) -> /AX_DIR1
- JP102 pad JP2_8: /SERVO8 -> unconnected-(JP102B-E19-PadJP2_8)
- JP102 pad JP2_9: unconnected-(JP102B-B19-PadJP2_9) -> /AX_DATA1
- Q101 pad 3: Net-(J113-Pin_1) -> Net-(J113-Pin_3)
- Q103 pad 3: Net-(J115-Pin_1) -> Net-(J115-Pin_3)
- Q104 pad 3: Net-(J118-Pin_1) -> Net-(J118-Pin_3)
- Q105 pad 3: Net-(J120-Pin_1) -> Net-(J120-Pin_3)
- Q106 pad 3: Net-(J121-Pin_1) -> Net-(J121-Pin_3)
- R113 pad 1: 3V3 -> +3V3
- R114 pad 2: Net-(J106-Pin_2) -> Net-(C114-Pad1)
- R115 pad 1: Net-(J106-Pin_2) -> Net-(C114-Pad1)
- R119 pad 2: /AX_DATA -> /AX_DATA1
- R122 pad 1: /AX_DATA -> /AX_DATA1
- R124 pad 1: /AX_DIR -> /AX_DIR1
- R127 pad 2: /AX_DATA -> /AX_DATA2
- R130 pad 1: /AX_DATA -> /AX_DATA2
- R132 pad 1: /AX_DIR -> /AX_DIR2
- R138 pad 2: Net-(J113-Pin_1) -> Net-(J113-Pin_3)
- R141 pad 2: Net-(J115-Pin_1) -> Net-(J115-Pin_3)
- R147 pad 2: Net-(J118-Pin_1) -> Net-(J118-Pin_3)
- R150 pad 2: Net-(J120-Pin_1) -> Net-(J120-Pin_3)
- R152 pad 2: Net-(J121-Pin_1) -> Net-(J121-Pin_3)
- U104 pad 5: /AX_DIR -> /AX_DIR1
- U105 pad 5: /AX_DIR -> /AX_DIR2
Routing:
- net +5V: track 4.93 -> 117.6 mm, vias 1 -> 7
- net +5V_SW: track 0.00 -> 83.9 mm, vias 0 -> 1
- net +5V_AO: track 35.9 -> 101.1 mm, vias 0 -> 10
- net GND: track 15.5 -> 75.9 mm, vias 7 -> 42
- net /AU: track 11.7 -> 68.8 mm, vias 0 -> 3
- net Net-(J121-Pin_3): track 0.00 -> 33.7 mm, vias 0 -> 3
- net /SERVO2: track 0.00 -> 29.3 mm, vias 0 -> 1
- net +3V3: track 11.4 -> 40.6 mm, vias 4 -> 19
- net /SERVO1: track 0.00 -> 27.7 mm, vias 0 -> 1
- net /WIFI_UART_TX: track 0.00 -> 26.0 mm, vias 0 -> 1
- net /SERVO4: track 0.00 -> 25.3 mm, vias 0 -> 1
- net /SERVO3: track 0.00 -> 24.9 mm, vias 0 -> 1
- net /LEDS: track 0.00 -> 24.7 mm, vias 0 -> 1
- net Net-(J120-Pin_3): track 0.00 -> 24.5 mm
- net Net-(J118-Pin_3): track 0.00 -> 22.5 mm, vias 0 -> 2
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- added copper zone on F.Cu, net +24V
- added copper zone on In2.Cu, net +3V3
- added copper zone on B.Cu, net +5V_AO
- added copper zone on F.Cu, net +5V_AO
- added copper zone on F.Cu, net +5V_SW
- added copper zone on B.Cu, net GND
- added copper zone on F.Cu, net GND
- added copper zone on In1.Cu, net GND
- added copper zone on F.Cu, net Net-(U101-SW)
- added copper zone on F.Cu, net Net-(U102-SW)
Other:
- copper layers 2 -> 4

Commit message: Vraiment finished
Parts:
- added D106: Red, PCM_JLCPCB:D_0603, F.Cu at (120.6, 91.0)
- added D107: Red, PCM_JLCPCB:D_0603, F.Cu at (171.3, 45.7)
- added D108: Red, PCM_JLCPCB:D_0603, F.Cu at (171.5, 98.2)
- added D109: Red, PCM_JLCPCB:D_0603, F.Cu at (121.6, 86.1)
- added D110: Red, PCM_JLCPCB:D_0603, F.Cu at (101.7, 78.7)
- added G***: LOGO, LOGO, F.Cu at (147.7, 66.2)
- added R153: 10kΩ, PCM_JLCPCB:R_0402, F.Cu at (121.9, 91.5)
- added R154: 1kΩ, PCM_JLCPCB:R_0402, F.Cu at (171.3, 47.1)
- added R155: 1kΩ, PCM_JLCPCB:R_0402, F.Cu at (171.5, 96.6)
- added R156: 1kΩ, PCM_JLCPCB:R_0402, F.Cu at (121.6, 83.5)
- added R157: 1kΩ, PCM_JLCPCB:R_0402, F.Cu at (103.7, 78.8)
- added TP102: TestPoint, TestPoint:TestPoint_THTPad_D1.0mm_Drill0.5mm, F.Cu at (131.9, 78.9)
- added TP103: TestPoint, TestPoint:TestPoint_THTPad_D1.0mm_Drill0.5mm, F.Cu at (111.5, 78.8)
- added TP104: TestPoint, TestPoint:TestPoint_THTPad_D1.0mm_Drill0.5mm, F.Cu at (172.7, 49.3)
- added TP105: TestPoint, TestPoint:TestPoint_THTPad_D1.0mm_Drill0.5mm, F.Cu at (172.0, 95.2)
Routing:
- net +5V: track 117.6 -> 139.0 mm, vias 7 -> 9
- net GND: track 75.9 -> 90.2 mm, vias 42 -> 44
- net +5V_SW: track 83.9 -> 88.3 mm
- net +5V_AO: track 101.1 -> 103.7 mm
- net Net-(D108-Pad2): track 0.00 -> 1.72 mm
- net Net-(D106-Pad2): track 0.00 -> 1.63 mm
- net Net-(D107-Pad2): track 0.00 -> 1.52 mm
- net +3V3: track 40.6 -> 42.0 mm
- net Net-(D110-Pad2): track 0.00 -> 1.38 mm
- net Net-(D109-Pad2): track 0.00 -> 1.31 mm
- net +24V: track 11.2 -> 12.1 mm
Other:
- board text added: "AU"
- board text added: "AX12"
- board text added: "B1"
- board text added: "B2"
- board text added: "B3"
- board text added: "CAN"
- board text added: "LIDAR"
- board text added: "Les Opossums"
- board text added: "SERVO"
- board text added: "TIR"
