File: ELE_MB_A1.kicad_sch (KiCad schematic)
At the start: 126 parts, among them J101 Conn_01x02, J102 Conn_01x02, J103 Conn_01x02, J104 Conn_01x02, J105 Conn_01x02, J106 Conn_01x02, J107 Conn_01x04, J108 Conn_01x03, J109 Conn_01x04, J110 Conn_01x03, J111 Conn_01x04, J112 Conn_01x04, J113 Conn_01x03, J114 Conn_01x04, J115 Conn_01x03, J116 Conn_01x04, J117 Conn_01x03, J118 Conn_01x03, J119 Conn_01x04, J120 Conn_01x03, J121 Conn_01x03, Q101 2N7002, Q102 SI2301CDS-T1-GE3, Q103 2N7002, Q104 2N7002, Q105 2N7002, Q106 2N7002, U101 TPS54302, U102 TPS54302, U103 SN65HVD230, U104 SN74LVC1T45DBV, U105 SN74LVC1T45DBV, U106 XIAO-ESP32-C3-DIP

Commit message: Finished board
Parts:
- added D105: B5818WS, PCM_JLCPCB:D_SOD-323, symbol PCM_JLCPCB-Diodes:Schottky,B5818WS
Connections:
- net 3V3 is gone; now on net +3V3: R113.1
- net SERVO6 is gone; now on net SERVO4: JP102.JP2_6 (F17)
- net AU: now also JP102.JP2_19 (G19); no longer JP102.JP2_21 (J18)
- net CAND: now also JP102.JP1_21 (T17); no longer JP102.JP1_1 (N17)
- net CANR: now also JP102.JP1_19 (V16); no longer JP102.JP1_2 (P18)
- net GND: now also J113.1 (Pin_1), J115.1 (Pin_1), J118.1 (Pin_1), J120.1 (Pin_1), J121.1 (Pin_1); no longer J113.3 (Pin_3), J115.3 (Pin_3), J118.3 (Pin_3), J120.3 (Pin_3), J121.3 (Pin_3)
- net LEDS: now also JP102.JP1_10 (Y19)
- net LIDAR_RX1: now also JP102.JP1_3 (R16); no longer JP102.JP1_5 (T16)
- net LIDAR_RX2: now also JP102.JP1_5 (T16); no longer JP102.JP1_7 (W18), JP102.JP2_10 (A20)
- net LIDAR_RX3: now also JP102.JP1_7 (W18); no longer JP102.JP1_8 (W19)
- net SERVO1: now also JP102.JP2_1 (L16); no longer JP102.JP2_2 (L17)
- net SERVO2: now also JP102.JP2_4 (G15); no longer JP102.JP2_1 (L16)
- net SERVO3: now also JP102.JP2_3 (H15); no longer JP102.JP2_4 (G15)
- net SERVO4: no longer JP102.JP2_3 (H15)
- net TIRETTE: now also JP102.JP2_27 (G17); no longer JP102.JP2_33 (F19)
- net WIFI_UART_RX: now also JP102.JP2_2 (L17)
- net WIFI_UART_TX: now also JP102.JP2_5 (F16)
- net at C114.1, R114.2, R115.1: now also D105.2; no longer J106.2 (Pin_2)
- net at Q104.3 (D), R147.2: now also J118.3 (Pin_3); no longer J118.1 (Pin_1)
- net at Q101.3 (D), R138.2: now also J113.3 (Pin_3); no longer J113.1 (Pin_1)
- net at Q103.3 (D), R141.2: now also J115.3 (Pin_3); no longer J115.1 (Pin_1)
- net at Q106.3 (D), R152.2: now also J121.3 (Pin_3); no longer J121.1 (Pin_1)
- net at Q105.3 (D), R150.2: now also J120.3 (Pin_3); no longer J120.1 (Pin_1)
- net AX_DIR2: now reaches JP102.JP2_13 (D19)
- net AX_DIR2: now also R132.1, U105.5 (DIR)
- net AX_DATA2: now reaches JP102.JP2_17 (H16)
- net AX_DATA2: now also R127.2, R130.1
- net AX_DIR1: now reaches JP102.JP2_7 (E18)
- net AX_DIR1: now also R124.1, U104.5 (DIR)
- net AX_DATA1: now reaches JP102.JP2_9 (B19)
- net AX_DATA1: now also R119.2, R122.1
- removed net AX_DATA: JP102.JP2_19 (G19), R119.2, R122.1, R127.2, R130.1
- removed net AX_DIR: JP102.JP2_40 (H20), R124.1, R132.1, U104.5 (DIR), U105.5 (DIR)
- net DIR1: no longer names the net of JP102.JP2_28 (G18)
- net DIR2: no longer names the net of JP102.JP2_34 (F20)
- net IO2: no longer names the net of JP102.JP2_26 (B20)
- net IO4: no longer names the net of JP102.JP2_24 (J16)
- net IO6: no longer names the net of JP102.JP2_22 (H18)
- net SERVO8: no longer names the net of JP102.JP2_8 (E19)
- net SPARE21: no longer names the net of JP102.JP2_18 (H17)
- net SPARE22: no longer names the net of JP102.JP2_16 (D18)
- net SPARE26: no longer names the net of JP102.JP2_14 (D20)
- net SPARE27: no longer names the net of JP102.JP2_20 (G20)
- net STP1: no longer names the net of JP102.JP2_32 (L20)
- net nEN_DRIVER2: no longer names the net of JP102.JP2_36 (M20)
- new net: D105.1, J106.2 (Pin_2)
- no-connect marks 12 -> 61
Other:
- note added: "24V Input"
- note added: "24V generates two 5V - AO (Always On, for LED, LIDARs and Wi-Fi) - NO AU - SW (Switched, for servoes) - AU Supplied by FPGA: - 3V3 Logic and Interfaces (Low Power) - 5V Logic and Interfaces (Low Power) I/Os: 3V3: - IN: Buttons (x3) - IN: AU (Emergency Stop) - IN: Tirette - INOUT: CAN - INOUT: Wi-Fi 5V: - IN: LIDARs - INOUT: AX12 (x2) - OUT: LEDs - OUT: Servos"
- note added: "5V Generation"
- note removed: "24V connected to ON/OFF, but not to emergency stop. Used to supply FPGA."
- note removed: "Power supply input"
- moved on the sheet: C114, J101, J121, JP102A, JP102B, Q106, R114, R115, R151, R152

Commit message: Vraiment finished
Parts:
- added D106, D107, D108, D109, D110: Red, PCM_JLCPCB:D_0603, symbol PCM_JLCPCB-Diodes:LED,0603,Red
- added R153: 10kΩ, PCM_JLCPCB:R_0402, symbol PCM_JLCPCB-Resistors:0402,10kΩ
- added R154, R155, R156, R157: 1kΩ, PCM_JLCPCB:R_0402, symbol PCM_JLCPCB-Resistors:0402,1kΩ
- added TP102, TP103, TP104, TP105: TestPoint, TestPoint:TestPoint_THTPad_D1.0mm_Drill0.5mm, symbol Connector:TestPoint
Connections:
- net +24V: now also R153.1
- net +3V3: now also R155.1, TP105.1
- net +5V: now also R154.1, TP104.1
- net +5V_AO: now also R156.1, TP102.1
- net +5V_SW: now also R157.1, TP103.1
- net GND: now also D106.1, D107.1, D108.1, D109.1, D110.1
- new net: D107.2, R154.2
- new net: D109.2, R156.2
- new net: D108.2, R155.2
- new net: D106.2, R153.2
- new net: D110.2, R157.2
Other:
- note added: "LEDs"
